File: Hardware/Charger/Pogocharge.kicad_pcb (KiCad board)
At the start: 2 copper layers, 245 x 200 mm, 30 parts, among them J1 Barrel_Jack_Switch, J10 90224-AS, J11 90224-AS, J12 90224-AS, J13 90224-AS, J15 90224-AS, J16 90224-AS, J17 90224-AS, J19 90224-AS, J20 90224-AS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

Commit message: fixing bug for charger
Routing:
- net +5V: track 111.0 -> 12.3 mm
Changed lines of the file:
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@@
   (segment (start 381.37 192) (end 381.39 191.98) (width 2) (layer "F.Cu") (net 1))
   (segment (start 376.35 189.01) (end 379.34 192) (width 2) (layer "F.Cu") (net 1))
-  (segment (start 376.35 90.37) (end 376.35 128.824) (width 2) (layer "F.Cu") (net 1))
   (segment (start 378.74 87.98) (end 376.35 90.37) (width 2) (layer "F.Cu") (net 1))
-  (segment (start 376.35 128.824) (end 376.35 189.01) (width 2) (layer "F.Cu") (net 1))
   (segment (start 182.475 143.76) (end 182.475 146.03) (width 0.25) (layer "F.Cu") (net 2))
   (segment (start 182.475 146.03) (end 182.375 146.13) (width 0.25) (layer "F.Cu") (net 2))
