File: Hardware/remote_leds_wall_strip/remote_leds_wall_strip.kicad_pcb (KiCad board)
At the start: 2 copper layers, 175 x 9 mm, 18 parts, among them J1 Conn_01x02_Male

Commit message: upgrade wall led strip from 20cm to 50cm
Parts:
- removed J1: Conn_01x02_Male, Connector_PinHeader_2.54mm:PinHeader_1x02_P2.54mm_Vertical
- added L11: VSMB3940X01-GS08, Footprints:LEDM3528X185N, F.Cu at (211.4, 95.3)
- added L12: VSMB3940X01-GS08, Footprints:LEDM3528X185N, F.Cu at (227.9, 95.3)
- added L13: VSMB3940X01-GS08, Footprints:LEDM3528X185N, F.Cu at (244.4, 95.3)
- added L14: VSMB3940X01-GS08, Footprints:LEDM3528X185N, F.Cu at (260.9, 95.3)
- added L15: VSMB3940X01-GS08, Footprints:LEDM3528X185N, F.Cu at (277.4, 95.3)
- added L16: VSMB3940X01-GS08, Footprints:LEDM3528X185N, F.Cu at (294.9, 95.3)
- added L17: VSMB3940X01-GS08, Footprints:LEDM3528X185N, F.Cu at (310.9, 95.3)
- added L18: VSMB3940X01-GS08, Footprints:LEDM3528X185N, F.Cu at (326.9, 95.3)
- added L19: VSMB3940X01-GS08, Footprints:LEDM3528X185N, F.Cu at (344.4, 95.3)
- added L20: VSMB3940X01-GS08, Footprints:LEDM3528X185N, F.Cu at (359.9, 95.3)
- added L21: VSMB3940X01-GS08, Footprints:LEDM3528X185N, F.Cu at (442.4, 95.3)
- added L22: VSMB3940X01-GS08, Footprints:LEDM3528X185N, F.Cu at (458.9, 95.3)
- added L23: VSMB3940X01-GS08, Footprints:LEDM3528X185N, F.Cu at (409.4, 95.3)
- added L24: VSMB3940X01-GS08, Footprints:LEDM3528X185N, F.Cu at (425.9, 95.3)
- added L25: VSMB3940X01-GS08, Footprints:LEDM3528X185N, F.Cu at (508.4, 95.3)
- added L26: VSMB3940X01-GS08, Footprints:LEDM3528X185N, F.Cu at (524.9, 95.3)
- added L27: VSMB3940X01-GS08, Footprints:LEDM3528X185N, F.Cu at (475.4, 95.3)
- added L28: VSMB3940X01-GS08, Footprints:LEDM3528X185N, F.Cu at (491.9, 95.3)
- added L29: VSMB3940X01-GS08, Footprints:LEDM3528X185N, F.Cu at (376.4, 95.3)
- added L30: VSMB3940X01-GS08, Footprints:LEDM3528X185N, F.Cu at (392.9, 95.3)
- added R10: 36, Resistor_SMD:R_0805_2012Metric_Pad1.20x1.40mm_HandSolder, F.Cu at (340.5, 94.8)
- added R11: 36, Resistor_SMD:R_0805_2012Metric_Pad1.20x1.40mm_HandSolder, F.Cu at (438.5, 94.8)
- added R12: 36, Resistor_SMD:R_0805_2012Metric_Pad1.20x1.40mm_HandSolder, F.Cu at (405.5, 94.8)
- added R13: 36, Resistor_SMD:R_0805_2012Metric_Pad1.20x1.40mm_HandSolder, F.Cu at (504.5, 94.8)
- added R14: 36, Resistor_SMD:R_0805_2012Metric_Pad1.20x1.40mm_HandSolder, F.Cu at (471.5, 94.8)
- added R15: 36, Resistor_SMD:R_0805_2012Metric_Pad1.20x1.40mm_HandSolder, F.Cu at (372.5, 94.8)
- added R6: 36, Resistor_SMD:R_0805_2012Metric_Pad1.20x1.40mm_HandSolder, F.Cu at (207.5, 94.8)
- added R7: 36, Resistor_SMD:R_0805_2012Metric_Pad1.20x1.40mm_HandSolder, F.Cu at (240.5, 94.8)
- added R8: 36, Resistor_SMD:R_0805_2012Metric_Pad1.20x1.40mm_HandSolder, F.Cu at (273.5, 94.8)
- added R9: 36, Resistor_SMD:R_0805_2012Metric_Pad1.20x1.40mm_HandSolder, F.Cu at (307.0, 94.8)
- added TP10: TestPoint, TestPoint:TestPoint_Pad_2.5x2.5mm, F.Cu at (233.0, 92.5)
- added TP11: TestPoint, TestPoint:TestPoint_Pad_2.5x2.5mm, F.Cu at (398.0, 98.0)
- added TP12: TestPoint, TestPoint:TestPoint_Pad_2.5x2.5mm, F.Cu at (266.0, 92.5)
- added TP13: TestPoint, TestPoint:TestPoint_Pad_2.5x2.5mm, F.Cu at (464.0, 98.0)
- added TP14: TestPoint, TestPoint:TestPoint_Pad_2.5x2.5mm, F.Cu at (32.9, 92.5)
- added TP15: TestPoint, TestPoint:TestPoint_Pad_2.5x2.5mm, F.Cu at (233.0, 98.0)
- added TP16: TestPoint, TestPoint:TestPoint_Pad_2.5x2.5mm, F.Cu at (464.0, 92.5)
- added TP17: TestPoint, TestPoint:TestPoint_Pad_2.5x2.5mm, F.Cu at (102.0, 98.0)
- added TP18: TestPoint, TestPoint:TestPoint_Pad_2.5x2.5mm, F.Cu at (69.5, 92.5)
- added TP19: TestPoint, TestPoint:TestPoint_Pad_2.5x2.5mm, F.Cu at (365.0, 98.0)
- added TP20: TestPoint, TestPoint:TestPoint_Pad_2.5x2.5mm, F.Cu at (365.0, 92.5)
- added TP21: TestPoint, TestPoint:TestPoint_Pad_2.5x2.5mm, F.Cu at (299.8, 98.0)
- added TP22: TestPoint, TestPoint:TestPoint_Pad_2.5x2.5mm, F.Cu at (332.0, 92.5)
- added TP23: TestPoint, TestPoint:TestPoint_Pad_2.5x2.5mm, F.Cu at (168.2, 98.0)
- added TP24: TestPoint, TestPoint:TestPoint_Pad_2.5x2.5mm, F.Cu at (168.2, 92.5)
- added TP25: TestPoint, TestPoint:TestPoint_Pad_2.5x2.5mm, F.Cu at (266.0, 98.0)
- added TP26: TestPoint, TestPoint:TestPoint_Pad_2.5x2.5mm, F.Cu at (299.8, 92.5)
- added TP27: TestPoint, TestPoint:TestPoint_Pad_2.5x2.5mm, F.Cu at (332.0, 98.0)
- added TP28: TestPoint, TestPoint:TestPoint_Pad_2.5x2.5mm, F.Cu at (398.0, 92.5)
- added TP3: TestPoint, TestPoint:TestPoint_Pad_2.5x2.5mm, F.Cu at (102.0, 92.5)
- added TP31: TestPoint, TestPoint:TestPoint_Pad_2.5x2.5mm, F.Cu at (497.0, 92.5)
- added TP32: TestPoint, TestPoint:TestPoint_Pad_2.5x2.5mm, F.Cu at (497.2, 98.0)
- added TP4: TestPoint, TestPoint:TestPoint_Pad_2.5x2.5mm, F.Cu at (135.2, 98.0)
- added TP5: TestPoint, TestPoint:TestPoint_Pad_2.5x2.5mm, F.Cu at (69.5, 98.0)
- added TP6: TestPoint, TestPoint:TestPoint_Pad_2.5x2.5mm, F.Cu at (135.2, 92.5)
- added TP7: TestPoint, TestPoint:TestPoint_Pad_2.5x2.5mm, F.Cu at (431.0, 98.0)
- added TP8: TestPoint, TestPoint:TestPoint_Pad_2.5x2.5mm, F.Cu at (431.0, 92.5)
- added TP9: TestPoint, TestPoint:TestPoint_Pad_2.5x2.5mm, F.Cu at (32.9, 98.0)
- moved R1 4.95 mm to (42.8, 94.8)
- moved L1 4.50 mm to (46.4, 95.3)
- moved R2 4.21 mm to (76.0, 94.8)
- moved L2 4.00 mm to (62.9, 95.3)
- moved R4 3.75 mm to (141.5, 94.8)
- moved L3 3.50 mm to (79.4, 95.3)
- moved L7 3.50 mm to (145.4, 95.3)
- moved R3 3.04 mm to (108.8, 94.8)
- moved L4 3.00 mm to (95.9, 95.3)
- moved L5 2.50 mm to (112.4, 95.3)
- moved L6 2.00 mm to (128.9, 95.3)
- moved R5 1.61 mm to (175.0, 94.8)
- moved L8 1.00 mm to (161.9, 95.3)
- moved TP1 0.89 mm to (201.5, 92.5)
- moved TP2 0.81 mm to (201.5, 98.0)
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Routing:
- net GND: track 180.6 -> 522.1 mm
- net VCC: track 180.8 -> 518.5 mm
- net Net-(L15-Pad1): track 0.00 -> 17.5 mm
- net Net-(L29-Pad1): track 0.00 -> 16.5 mm
- net Net-(L27-Pad1): track 0.00 -> 16.5 mm
- net Net-(L25-Pad1): track 0.00 -> 16.5 mm
- net Net-(L23-Pad1): track 0.00 -> 16.5 mm
- net Net-(L21-Pad1): track 0.00 -> 16.5 mm
- net Net-(L11-Pad1): track 0.00 -> 16.5 mm
- net Net-(L13-Pad1): track 0.00 -> 16.5 mm
- net Net-(L17-Pad1): track 0.00 -> 16.0 mm
- net Net-(L19-Pad1): track 0.00 -> 15.5 mm
- net Net-(L13-Pad2): track 0.00 -> 3.90 mm
- net Net-(L11-Pad2): track 0.00 -> 3.90 mm
- net Net-(L29-Pad2): track 0.00 -> 3.90 mm
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Other:
- board size 175 x 9 mm -> 500 x 9 mm

Commit message: changing the size of the strip led from 50 to 30cm
Parts:
- removed L19, L20, L21, L22, L23, L24, L25, L26, L27, L28, L29, L30: VSMB3940X01-GS08, Footprints:LEDM3528X185N
- removed R10, R11, R12, R13, R14, R15: 36, Resistor_SMD:R_0805_2012Metric_Pad1.20x1.40mm_HandSolder
- removed TP11, TP13, TP16, TP19, TP20, TP28, TP31, TP32, TP7, TP8: TestPoint, TestPoint:TestPoint_Pad_2.5x2.5mm
Routing:
- net GND: track 522.1 -> 317.7 mm
- net VCC: track 518.5 -> 327.7 mm
- net Net-(L29-Pad1): track 16.5 -> 0.00 mm
- net Net-(L27-Pad1): track 16.5 -> 0.00 mm
- net Net-(L25-Pad1): track 16.5 -> 0.00 mm
- net Net-(L23-Pad1): track 16.5 -> 0.00 mm
- net Net-(L21-Pad1): track 16.5 -> 0.00 mm
- net Net-(L19-Pad1): track 15.5 -> 0.00 mm
- net Net-(L29-Pad2): track 3.90 -> 0.00 mm
- net Net-(L27-Pad2): track 3.90 -> 0.00 mm
- net Net-(L25-Pad2): track 3.90 -> 0.00 mm
- net Net-(L23-Pad2): track 3.90 -> 0.00 mm
- net Net-(L21-Pad2): track 3.90 -> 0.00 mm
- net Net-(L19-Pad2): track 3.90 -> 0.00 mm
Other:
- board size 500 x 9 mm -> 305 x 9 mm
