File: Hardware/remote_leds_wall_ctrl/remote_leds_wall_ctrl.kicad_pcb (KiCad board)
At the start: 2 copper layers, 47 x 31 mm, 17 parts, among them J1 Conn_01x03_Male, J2 Conn_01x02_Female, Q2 ZXMN3A14F, U2 mcp1407

Commit message: change transistor in wall crtl
Parts:
- Q2: value ZXMN3A14F -> BSR802NL6327HTSA1
- RV1: value Potentiometer -> 100
Changed lines of the file:
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@@
   (net 1 "VCC")
   (net 2 "GND")
-  (net 3 "Net-(Q2-Pad3)")
+  (net 3 "Net-(J2-Pad2)")
   (net 4 "Net-(Q2-Pad1)")
   (net 5 "unconnected-(U2-Pad3)")
@@
       (effects (font (size 1 1) (thickness 0.15)))
     )
-    (fp_text value "ZXMN3A14F" (at 0 2.4) (layer "F.Fab") hide
+    (fp_text value "BSR802NL6327HTSA1" (at 0 2.4) (layer "F.Fab") hide
       (effects (font (size 1 1) (thickness 0.15)))
     )
@@
       (net 2 "GND") (pinfunction "S") (pintype "passive"))
     (pad "3" smd roundrect (at 0.9375 0) (size 1.475 0.6) (layers "F.Cu" "F.Paste" "F.Mask") (roundrect_rratio 0.25)
-      (net 3 "Net-(Q2-Pad3)") (pinfunction "D") (pintype "passive"))
+      (net 3 "Net-(J2-Pad2)") (pinfunction "D") (pintype "passive"))
     (model "${KICAD6_3DMODEL_DIR}/Package_TO_SOT_SMD.3dshapes/SOT-23.wrl"
       (offset (xyz 0 0 0))
@@
       (net 7 "Net-(J2-Pad1)") (pinfunction "Pin_1") (pintype "passive"))
     (pad "2" thru_hole oval (at 0 2.54) (size 1.7 1.7) (drill 1) (layers *.Cu *.Mask)
-      (net 3 "Net-(Q2-Pad3)") (pinfunction "Pin_2") (pintype "passive"))
+      (net 3 "Net-(J2-Pad2)") (pinfunction "Pin_2") (pintype "passive"))
     (model "${KICAD6_3DMODEL_DIR}/Connector_PinHeader_2.54mm.3dshapes/PinHeader_1x02_P2.54mm_Vertical.wrl"
       (offset (xyz 0 0 0))
@@
       (effects (font (size 1 1) (thickness 0.15)))
     )
-    (fp_text value "Potentiometer" (at -2.75 2.525 180) (layer "F.Fab") hide
+    (fp_text value "100" (at -2.75 2.525 180) (layer "F.Fab") hide
       (effects (font (size 1 1) (thickness 0.15)))
     )
