File: Hardware/remote_leds_wall_ctrl/remote_leds_wall_ctrl.kicad_sch (KiCad schematic)
At the start: 11 parts, among them J1 Conn_01x03_Male, J2 Conn_01x02_Female, Q2 ZXMN3A14F, U2 mcp1407

Commit message: update resistance values
Parts:
- RV1: value R_Potentiometer -> 100
Changed lines of the file:
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@@
       (effects (font (size 1.27 1.27)) (justify right))
     )
-    (property "Value" "R_Potentiometer" (id 1) (at 167.64 45.7199 0)
+    (property "Value" "100" (id 1) (at 167.64 45.7199 0)
       (effects (font (size 1.27 1.27)) (justify right))
     )
@@
     )
     (path "/aabf9e25-f19a-483c-b34c-a24443ca1f71"
-      (reference "RV1") (unit 1) (value "R_Potentiometer") (footprint "Connector_PinHeader_2.54mm:PinHeader_1x03_P2.54mm_Vertical")
+      (reference "RV1") (unit 1) (value "100") (footprint "Connector_PinHeader_2.54mm:PinHeader_1x03_P2.54mm_Vertical")
     )
     (path "/dc03aa88-db40-4ba7-9f35-1acc4d16523f"

Commit message: change transistor in wall crtl
Parts:
- Q2: value ZXMN3A14F -> BSR802NL6327HTSA1
Changed lines of the file:
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@@
       (effects (font (size 1.27 1.27)) (justify left))
     )
-    (property "Value" "ZXMN3A14F" (id 1) (at 173.99 99.0599 0)
+    (property "Value" "BSR802NL6327HTSA1" (id 1) (at 173.99 99.0599 0)
       (effects (font (size 1.27 1.27)) (justify left))
     )
@@
       (effects (font (size 1.27 1.27) italic) (justify left) hide)
     )
-    (property "Datasheet" "http://www.diodes.com/assets/Datasheets/ZXMN3A14F.pdf" (id 3) (at 167.64 97.79 0)
+    (property "Datasheet" "https://www.mouser.fr/ProductDetail/Infineon-Technologies/BSR802NL6327HTSA1?qs=K00xGehIljs0LeKKuwlBqA%3D%3D&srsltid=AfmBOorBgLAkgF7Xqp9mXzJpMe1H2BGHlg6ZcHs-kYA68t-aJlhnifkq" (id 3) (at 167.64 97.79 0)
       (effects (font (size 1.27 1.27)) (justify left) hide)
     )
@@
     )
     (path "/13b09df4-ad66-472e-abc0-6d9536cf2c68"
-      (reference "Q2") (unit 1) (value "ZXMN3A14F") (footprint "Package_TO_SOT_SMD:SOT-23")
+      (reference "Q2") (unit 1) (value "BSR802NL6327HTSA1") (footprint "Package_TO_SOT_SMD:SOT-23")
     )
     (path "/c69753b9-9301-45db-a6ba-e9b8e78cee91"
