File: Hardware/Belly/motor_ctrl.kicad_sch (KiCad schematic)
At the start: 5 parts, among them U1 DRV8837C

Commit message: adding belly v3
Parts:
- M1: value (none) -> Motor_DC; footprint (none) -> MyFootprints:Vibrating_5x6mm_DC_motor
- R3: footprint (none) -> Resistor_SMD:R_0805_2012Metric
- U1: footprint Package_SON:WSON-8-1EP_2x2mm_P0.5mm_EP0.9x1.6mm -> Footprints:WSON-8-1EP_2x2mm_P0.5mm_EP0.9x1.6mm; symbol Driver_Motor:DRV8837C -> drv8837c:DRV8837C
Changed lines of the file:
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@@
   (junction (at 155.575 74.295) (diameter 0) (color 0 0 0 0)
   )
-  (wire (pts (xy 140.335 102.235) (xy 151.765 102.235))
-    (stroke (width 0) (type default) (color 0 0 0 0))
-  )
   (wire (pts (xy 165.1 70.485) (xy 165.1 74.295))
     (stroke (width 0) (type default) (color 0 0 0 0))
@@
     (stroke (width 0) (type default) (color 0 0 0 0))
   )
-  (wire (pts (xy 140.335 104.775) (xy 151.765 104.775))
-    (stroke (width 0) (type default) (color 0 0 0 0))
-  )
   (wire (pts (xy 181.61 109.855) (xy 181.61 108.585))
     (stroke (width 0) (type default) (color 0 0 0 0))
@@
     (stroke (width 0) (type default) (color 0 0 0 0))
   )
+  (wire (pts (xy 130.175 99.695) (xy 151.765 99.695))
+    (stroke (width 0) (type default) (color 0 0 0 0))
+  )
   (wire (pts (xy 155.575 74.295) (xy 145.415 74.295))
     (stroke (width 0) (type default) (color 0 0 0 0))
@@
     (stroke (width 0) (type default) (color 0 0 0 0))
   )
+  (wire (pts (xy 130.175 102.235) (xy 151.765 102.235))
+    (stroke (width 0) (type default) (color 0 0 0 0))
+  )
   (wire (pts (xy 181.61 94.615) (xy 181.61 95.885))
     (stroke (width 0) (type default) (color 0 0 0 0))
   )
-  (wire (pts (xy 140.335 99.695) (xy 151.765 99.695))
+  (wire (pts (xy 130.175 104.775) (xy 151.765 104.775))
     (stroke (width 0) (type default) (color 0 0 0 0))
   )
@@
     (stroke (width 0) (type default) (color 0 0 0 0))
   )
-  (hierarchical_label "Motor_sleep" (shape input) (at 140.335 99.695 180)
+  (hierarchical_label "Motor_sleep" (shape input) (at 130.175 99.695 180)
     (effects (font (size 1.27 1.27)) (justify right))
   )
-  (hierarchical_label "Motor_IN2" (shape input) (at 140.335 104.775 180)
+  (hierarchical_label "Motor_IN2" (shape input) (at 130.175 104.775 180)
     (effects (font (size 1.27 1.27)) (justify right))
   )
-  (hierarchical_label "Motor_IN1" (shape input) (at 140.335 102.235 180)
+  (hierarchical_label "Motor_IN1" (shape input) (at 130.175 102.235 180)
     (effects (font (size 1.27 1.27)) (justify right))
   )
@@
       (effects (font (size 1.27 1.27)) (justify left))
     )
-    (property "Value" "" (id 1) (at 185.6232 103.378 0)
-      (effects (font (size 1.27 1.27)) (justify left))
-    )
-    (property "Footprint" "" (id 2) (at 181.61 103.251 0)
+    (property "Value" "Motor_DC" (id 1) (at 185.6232 103.378 0)
+      (effects (font (size 1.27 1.27)) (justify left))
+    )
+    (property "Footprint" "MyFootprints:Vibrating_5x6mm_DC_motor" (id 2) (at 181.61 103.251 0)
       (effects (font (size 1.27 1.27)) hide)
     )
@@
     (property "Reference" "R3" (id 0) (at 160.655 64.77 90))
     (property "Value" "0" (id 1) (at 160.655 67.31 90))
-    (property "Footprint" "" (id 2) (at 160.655 72.263 90)
+    (property "Footprint" "Resistor_SMD:R_0805_2012Metric" (id 2) (at 160.655 72.263 90)
       (effects (font (size 1.27 1.27)) hide)
     )
@@
     (pin "1")
   )
-  (symbol (lib_id "Driver_Motor:DRV8837C") (at 161.925 102.235 0) (unit 1)
+  (symbol (lib_id "drv8837c:DRV8837C") (at 161.925 102.235 0) (unit 1)
     (in_bom yes) (on_board yes) (fields_autoplaced)
     (property "Reference" "U1" (id 0) (at 163.9444 115.57 0)
@@
       (effects (font (size 1.27 1.27)) (justify left))
     )
-    (property "Footprint" "Package_SON:WSON-8-1EP_2x2mm_P0.5mm_EP0.9x1.6mm" (id 2) (at 161.925 123.825 0)
-      (effects (font (size 1.27 1.27)) hide)
-    )
+    (property "Footprint" "Footprints:WSON-8-1EP_2x2mm_P0.5mm_EP0.9x1.6mm" (id 2) (at 161.925 123.825 0)
+      (effects (font (size 1.27 1.27)) hide)
+    )
